Commit message: 新增dual arm ik fk tr

File: description/tiangong_description/urdf/tiangong2_EVT_V2.urdf (robot description, URDF)
Before this commit: robot humanoid, 35 links, 34 joints
Joints:
- removed joint fixed_to_world
- added joint world_joint: type fixed, parent world, child pelvis, origin xyz=0 0 1.2 rpy=0 0 0
